File: Hardware/Connected-OldtimerHardware/_saved_Connected-OldtimerHardware.sch (KiCad schematic (older format))
At the start: 16 parts, among them J1 CAN_Bus_Connector, J2 MainConnector, J3 NextionConnector, Q1 2N3906, U1 ParticleElectron, U2 TSR_2-2450, U3 CANTranceiverModule, U4 AdafruitFRAM, U5 AdafruitUltimateGPS, U6 MotionSensor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

Commit message: completed footprints
Parts:
- U3: footprint (none) -> heathsfootprints:CAN_Tranceiver_Module
- U4: footprint (none) -> heathsfootprints:Adafruit_I2C_FRAM
- U5: footprint (none) -> heathsfootprints:AdafruitUltimateGPS
Changed lines of the file:
@@
 F 0 "U3" H 4977 1446 50  0000 L CNN
 F 1 "CANTranceiverModule" H 4977 1355 50  0000 L CNN
-F 2 "" H 4950 1300 50  0001 C CNN
+F 2 "heathsfootprints:CAN_Tranceiver_Module" H 4950 1300 50  0001 C CNN
 F 3 "" H 4950 1300 50  0001 C CNN
 	1    4950 1300
@@
 F 0 "U4" H 5078 2746 50  0000 L CNN
 F 1 "AdafruitFRAM" H 5078 2655 50  0000 L CNN
-F 2 "" H 4600 2800 50  0001 C CNN
+F 2 "heathsfootprints:Adafruit_I2C_FRAM" H 4600 2800 50  0001 C CNN
 F 3 "" H 4600 2800 50  0001 C CNN
 	1    4600 2800
@@
 F 0 "U5" H 5127 4771 50  0000 L CNN
 F 1 "AdafruitUltimateGPS" H 5127 4680 50  0000 L CNN
-F 2 "" H 4750 4700 50  0001 C CNN
+F 2 "heathsfootprints:AdafruitUltimateGPS" H 4750 4700 50  0001 C CNN
 F 3 "" H 4750 4700 50  0001 C CNN
 	1    4750 4700
